File: Potentiostat_LMP91002_breakout/Potentiostat_LMP91002_breakout.kicad_pcb (KiCad board)
At the start: 2 copper layers, 25.4 x 22.9 mm, 3 parts, among them P1 CONN_01X07, P2 CONN_01X07, U1 LMP91002

Commit message: added a bunch of stuff
Routing:
- net WE: track 7.33 -> 7.83 mm
- net VREF: track 6.49 -> 6.99 mm
- net VOUT: track 9.55 -> 10.1 mm
- net SDA: track 6.49 -> 6.99 mm
- net SCL: track 7.33 -> 7.83 mm
- net RE: track 8.92 -> 9.42 mm
- net MENB: track 8.92 -> 9.42 mm
- net CE: track 9.55 -> 10.1 mm
- net C2: track 8.92 -> 9.42 mm
- net C1: track 7.33 -> 7.83 mm
- net +3V3: track 8.92 -> 9.42 mm
Other:
- board text added: "1"
- board text added: "14"
- board text added: "CE"
- board text added: "GND"
- board text added: "Vout"
