File: Voltage_Regulator_MCP1700_breakout/Voltage_Regulator_MCP1700_breakout.sch (KiCad schematic (older format))
At the start: 2 parts, among them P1 CONN_01X03, U1 MCP1700

Commit message: added SPEC and SMM-102-02-S-S
Parts:
- P1: footprint (none) -> Socket_Strips:Socket_Strip_Straight_1x03
- U1: footprint (none) -> scintilla:MCP1700
Changed lines of the file:
@@
 F 0 "U1" H 5150 3200 60  0000 C CNN
 F 1 "MCP1700" H 4800 3800 60  0000 C CNN
-F 2 "" H 4800 3600 60  0001 C CNN
+F 2 "scintilla:MCP1700" H 4800 3600 60  0001 C CNN
 F 3 "" H 4800 3600 60  0001 C CNN
 	1    4800 3650
@@
 F 0 "P1" H 3300 3800 50  0000 C CNN
 F 1 "CONN_01X03" V 3400 3600 50  0000 C CNN
-F 2 "" H 3300 3600 50  0000 C CNN
+F 2 "Socket_Strips:Socket_Strip_Straight_1x03" H 3300 3600 50  0001 C CNN
 F 3 "" H 3300 3600 50  0000 C CNN
 	1    3300 3600
