File: ESP-12F_flash_with_cutout/ESP-12F_flash_with_cutout.sch (KiCad schematic (older format))
At the start: 11 parts, among them P1 CONN_01X12, P2 CONN_01X04, P3 CONN_01X03, P4 CONN_01X02, U1 ESP-12F

Commit message: fix for esp-12f
Parts:
- U1: footprint scintilla:ESP-12F -> (none)
Changed lines of the file:
@@
 $Comp
 L ESP-12F U1
-U 1 1 57C9FA90
+U 1 1 57C9FDC0
 P 6100 3500
 F 0 "U1" H 6100 3400 50  0000 C CNN
 F 1 "ESP-12F" H 6100 3600 50  0000 C CNN
-F 2 "scintilla:ESP-12F" H 6100 3500 50  0001 C CNN
+F 2 "" H 6100 3500 50  0001 C CNN
 F 3 "" H 6100 3500 50  0001 C CNN
 	1    6100 3500
