File: Battery_subsystem/Battery_subsystem.sch (KiCad schematic (older format))
At the start: 7 parts, among them U1 LTC4060, U2 MJD210

Commit message: added battery subsystem
Parts:
- removed BT1: Battery, symbol Battery
- added P1: CONN_01X02, Socket_Strips:Socket_Strip_Straight_1x02, symbol CONN_01X02
- added U3: 36-1022-ND, scintilla:36-1022-ND, symbol 36-1022-ND
- added U4: 609-4613-6-ND, scintilla:609-4613-6-ND, symbol 609-4613-6-ND
- C1: footprint (none) -> Capacitors_SMD:C_0805
- D1: footprint (none) -> LEDs:LED_0805
- R2, R3: footprint (none) -> Resistors_SMD:R_0805
- U1: footprint (none) -> scintilla:LTC4060
- U2: footprint (none) -> scintilla:MJD210
Connections:
- net +5V: now also U1.9 (SEL0), U4.1 (VCC); no longer U1.10 (SEL1)
- net BAT: now also P1.2 (P2), U3.1 (VOUT)
- net GND: now also U1.10 (SEL1), P1.1 (P1), U3.2 (GND), U4.5 (GND); no longer U1.9 (SEL0)
- new net: U3.3 (GND_POS), U3.4 (VOUT_NEG)
- no-connect marks 2 -> 4
Changed lines of the file:
@@
 LIBS:valves
 LIBS:scintilla
+LIBS:Battery_subsystem-cache
 EELAYER 25 0
 EELAYER END
@@
 F 0 "U1" H 6400 2800 60  0000 C CNN
 F 1 "LTC4060" H 5850 3650 60  0000 C CNN
-F 2 "" H 5850 3650 60  0000 C CNN
+F 2 "scintilla:LTC4060" H 5850 3650 60  0001 C CNN
 F 3 "" H 5850 3650 60  0000 C CNN
 	1    5850 3650
@@
 F 0 "U2" H 9100 2800 60  0000 C CNN
 F 1 "MJD210" H 8750 3450 60  0000 C CNN
-F 2 "" H 8750 3350 60  0000 C CNN
+F 2 "scintilla:MJD210" H 8750 3350 60  0001 C CNN
 F 3 "" H 8750 3350 60  0000 C CNN
 	1    8750 3350
@@
 Wire Wire Line
 	6650 3450 6800 3450
-$Comp
-L PWR_FLAG #FLG03
-U 1 1 57AE3A74
-P 3250 2750
-F 0 "#FLG03" H 3250 2845 50  0001 C CNN
-F 1 "PWR_FLAG" H 3250 2930 50  0000 C CNN
-F 2 "" H 3250 2750 50  0000 C CNN
-F 3 "" H 3250 2750 50  0000 C CNN
-	1    3250 2750
-	1    0    0    -1
-$EndComp
-$Comp
-L PWR_FLAG #FLG04
-U 1 1 57AE3A8E
-P 3250 3450
-F 0 "#FLG04" H 3250 3545 50  0001 C CNN
-F 1 "PWR_FLAG" H 3250 3630 50  0000 C CNN
-F 2 "" H 3250 3450 50  0000 C CNN
-F 3 "" H 3250 3450 50  0000 C CNN
-	1    3250 3450
-	1    0    0    -1
-$EndComp
-Wire Wire Line
-	3250 3450 3250 3550
-Wire Wire Line
-	3250 3550 3600 3550
 Wire Wire Line
 	3600 3550 3600 3400
@@
 	6650 3850 6800 3850
 Text GLabel 6800 4050 2    60   Input ~ 0
-GND
-Text GLabel 6800 3850 2    60   Input ~ 0
 Vin
 Text GLabel 6800 4250 2    60   Input ~ 0
 Vin
-Wire Wire Line
-	3250 2750 3250 2950
-Wire Wire Line
-	3250 2950 3800 2950
 Wire Wire Line
 	3650 2950 3650 2750
@@
 F 0 "R2" V 5830 1100 50  0000 C CNN
 F 1 "330" V 5750 1100 50  0000 C CNN
-F 2 "" V 5680 1100 50  0000 C CNN
+F 2 "Resistors_SMD:R_0805" V 5680 1100 50  0001 C CNN
 F 3 "" H 5750 1100 50  0000 C CNN
 	1    5750 1100
@@
 F 0 "D1" H 5750 1700 50  0000 C CNN
 F 1 "LED" H 5750 1500 50  0000 C CNN
-F 2 "" H 5750 1600 50  0000 C CNN
+F 2 "LEDs:LED_0805" H 5750 1600 50  0001 C CNN
 F 3 "" H 5750 1600 50  0000 C CNN
 	1    5750 1600
@@
 F 0 "R3" V 6980 1100 50  0000 C CNN
 F 1 "698" V 6900 1100 50  0000 C CNN
-F 2 "" V 6830 1100 50  0000 C CNN
+F 2 "Resistors_SMD:R_0805" V 6830 1100 50  0001 C CNN
 F 3 "" H 6900 1100 50  0000 C CNN
 	1    6900 1100
@@
 F 0 "C1" H 7775 1500 50  0000 L CNN
 F 1 "1.5n" H 7775 1300 50  0000 L CNN
-F 2 "" H 7788 1250 50  0000 C CNN
+F 2 "Capacitors_SMD:C_0805" H 7788 1250 50  0001 C CNN
 F 3 "" H 7750 1400 50  0000 C CNN
 	1    7750 1400
@@
 Text GLabel 8000 3550 0    60   Input ~ 0
 BAT
-$Comp
-L Battery BT1
-U 1 1 57AE46D9
-P 8050 4800
-F 0 "BT1" H 8150 4850 50  0000 L CNN
-F 1 "Battery" H 8150 4750 50  0000 L CNN
-F 2 "" V 8050 4840 50  0000 C CNN
-F 3 "" V 8050 4840 50  0000 C CNN
-	1    8050 4800
-	1    0    0    -1
-$EndComp
 Wire Wire Line
 	8050 4650 8050 4500
@@
 Text GLabel 4900 4250 0    60   Input ~ 0
 PROG
+$Comp
+L 609-4613-6-ND U4
+U 1 1 57D8B0DA
+P 3500 1450
+F 0 "U4" H 3850 1000 60  0000 C CNN
+F 1 "609-4613-6-ND" H 3500 1450 60  0000 C CNN
+F 2 "scintilla:609-4613-6-ND" H 3500 1450 60  0001 C CNN
+F 3 "" H 3500 1450 60  0001 C CNN
+	1    3500 1450
+	1    0    0    -1
+$EndComp
+Wire Wire Line
+	3500 2050 3700 2050
+Text GLabel 3700 2050 2    60   Input ~ 0
+GND
+NoConn ~ 4100 1600
+NoConn ~ 4100 1300
+Wire Wire Line
+	3500 850  3700 850
+Text GLabel 3700 850  2    60   Input ~ 0
+Vin
+Wire Wire Line
+	3800 2950 3650 2950
+$Comp
+L CONN_01X02 P1
+U 1 1 57D8BA11
+P 3200 4500
+F 0 "P1" H 3200 4650 50  0000 C CNN
+F 1 "CONN_01X02" V 3300 4500 50  0000 C CNN
+F 2 "Socket_Strips:Socket_Strip_Straight_1x02" H 3200 4500 50  0001 C CNN
+F 3 "" H 3200 4500 50  0000 C CNN
+	1    3200 4500
+	-1   0    0    1
+$EndComp
+Wire Wire Line
+	3400 4450 3400 4400
+Wire Wire Line
+	3400 4400 3450 4400
+Wire Wire Line
+	3400 4550 3400 4600
+Wire Wire Line
+	3400 4600 3450 4600
+Text GLabel 3450 4400 2    60   Input ~ 0
+BAT
+Text GLabel 3450 4600 2    60   Input ~ 0
+GND
+Wire Wire Line
+	6950 4650 6950 4950
+$Comp
+L 36-1022-ND U3
+U 1 1 57D96E3E
+P 7500 4800
+F 0 "U3" H 7800 4400 60  0000 C CNN
+F 1 "36-1022-ND" H 7500 4800 60  0000 C CNN
+F 2 "scintilla:36-1022-ND" H 7500 4800 60  0001 C CNN
+F 3 "" H 7500 4800 60  0001 C CNN
+	1    7500 4800
+	1    0    0    -1
+$EndComp
+Text GLabel 6800 3850 2    60   Input ~ 0
+GND
 $EndSCHEMATC
