File: Battery_subsystem/Battery_subsystem.kicad_pcb (KiCad board)
At the start: 2 copper layers, 35 x 70 mm, 9 parts, among them P1 CONN_01X02, U1 LTC4060, U2 MJD210, U3 36-1022-ND, U4 609-4613-6-ND

Commit message: added humidity sensor
Parts:
- added REF**: VIA-1.55mm-0.55mm, scintilla:VIA-1.55mm-0.55mm, F.Cu at (150.0, 70.0)
Routing:
- net GND: track 25.6 -> 43.8 mm
- net BAT: track 50.7 -> 51.4 mm
Other:
- net class Default: trace_width 0.35 -> 0.45
- rule trace_min: 0.35 -> 0.45
